File: P2I.kicad_pcb (KiCad board)
At the start: 2 copper layers, 68.5 x 50 mm, 30 parts, among them J1 Conn_01x02_Socket, J22 Conn_01x10_Socket, J23 Conn_01x20_Socket, U1 LM741CN_NOPB, U10 LM741CN_NOPB, U2 LM741CN_NOPB, U3 LM741CN_NOPB, U4 LM741CN_NOPB, U5 LM741CN_NOPB, U6 LM741CN_NOPB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

Commit message: Update
Parts:
- removed J1: Conn_01x02_Socket, Connector_PinSocket_1.27mm:PinSocket_1x02_P1.27mm_Vertical
- removed J22: Conn_01x10_Socket, Connector_PinSocket_1.27mm:PinSocket_1x10_P1.27mm_Vertical
- added J2: Conn_01x14_Socket, Connector_PinSocket_2.54mm:PinSocket_1x14_P2.54mm_Vertical, F.Cu at (201.0, 112.0)
- added J3: Conn_01x14_Socket, Connector_PinSocket_2.54mm:PinSocket_1x14_P2.54mm_Vertical, F.Cu at (180.7, 112.0)
- added J4: Conn_01x05_Socket, Connector_PinSocket_2.54mm:PinSocket_1x05_P2.54mm_Vertical, F.Cu at (161.3, 74.5)
- added VR16: T93YA104KT20, KiCad:T93YA5K10, F.Cu at (146.8, 109.0)
- added VR17: T93YA104KT20, KiCad:T93YA5K10, F.Cu at (171.8, 84.0)
- added VR18: T93YA104KT20, KiCad:T93YA5K10, F.Cu at (171.8, 96.0)
- added VR19: T93YA104KT20, KiCad:T93YA5K10, F.Cu at (171.8, 108.0)
- added VR20: T93YA104KT20, KiCad:T93YA5K10, F.Cu at (122.3, 114.0)
- C1, C2: footprint Connector_PinSocket_1.27mm:PinSocket_1x02_P1.27mm_Vertical -> Connector_PinSocket_2.54mm:PinSocket_1x02_P2.54mm_Vertical
- J23: footprint Connector_PinSocket_1.27mm:PinSocket_1x20_P1.27mm_Vertical -> Connector_PinSocket_2.54mm:PinSocket_1x20_P2.54mm_Vertical
- moved C2 69.2 mm to (193.5, 118.0)
- moved C1 59.8 mm to (184.0, 118.0)
- moved VR11 41.5 mm to (129.7, 108.9)
- moved U6 41.5 mm to (138.2, 108.9)
- moved U4 41.5 mm to (137.9, 84.4)
- moved U5 41.5 mm to (137.9, 96.4)
- moved VR1 41.5 mm to (104.3, 102.0)
- moved VR12 41.5 mm to (154.2, 84.0)
- moved VR13 41.5 mm to (154.3, 96.0)
- moved VR3 41.5 mm to (104.5, 90.0)
- moved VR6 41.5 mm to (121.8, 78.0)
- moved VR7 41.5 mm to (129.4, 83.9)
- moved VR9 41.5 mm to (129.4, 95.9)
- moved U1 41.5 mm to (113.0, 102.5)
- moved U10 41.5 mm to (113.5, 114.5)
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Connections:
- U10 pad 3: GND -> Net-(U10-NON-INV_INPUT)
- U6 pad 3: GND -> Net-(U6-NON-INV_INPUT)
- U7 pad 3: GND -> Net-(U7-NON-INV_INPUT)
- U8 pad 3: GND -> Net-(U8-NON-INV_INPUT)
- U9 pad 3: GND -> Net-(U9-NON-INV_INPUT)
Routing:
- net +5V: track 337.2 -> 455.8 mm
- net /A10: track 135.1 -> 153.3 mm
- net Net-(U10-NON-INV_INPUT): track 0.00 -> 11.4 mm
- net /Force1: track 39.8 -> 47.5 mm
- net /Flex2: track 55.5 -> 49.1 mm
- net Net-(U8-NON-INV_INPUT): track 0.00 -> 5.79 mm
- net Net-(U9-NON-INV_INPUT): track 0.00 -> 5.70 mm
- net /Flex5: track 56.0 -> 61.7 mm
- net Net-(U7-NON-INV_INPUT): track 0.00 -> 5.54 mm
- net /Flex3: track 41.4 -> 36.0 mm
- net /Flex4: track 27.3 -> 22.0 mm
- net Net-(U6-NON-INV_INPUT): track 0.00 -> 5.24 mm
- net /Force2: track 46.1 -> 50.9 mm
- net /Force3: track 59.0 -> 63.3 mm
- net /A9: track 61.8 -> 65.5 mm
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Other:
- board size 68.5 x 50 mm -> 105 x 50 mm
