File: P2I.kicad_sch (KiCad schematic)
At the start: 30 parts, among them J1 Conn_01x02_Socket, J22 Conn_01x10_Socket, J23 Conn_01x20_Socket, U1 LM741CN_NOPB, U10 LM741CN_NOPB, U2 LM741CN_NOPB, U3 LM741CN_NOPB, U4 LM741CN_NOPB, U5 LM741CN_NOPB, U6 LM741CN_NOPB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

Commit message: Update
Parts:
- removed J1: Conn_01x02_Socket, Connector_PinSocket_1.27mm:PinSocket_1x02_P1.27mm_Vertical, symbol Connector:Conn_01x02_Socket
- removed J22: Conn_01x10_Socket, Connector_PinSocket_1.27mm:PinSocket_1x10_P1.27mm_Vertical, symbol Connector:Conn_01x10_Socket
- added J2, J3: Conn_01x14_Socket, Connector_PinSocket_2.54mm:PinSocket_1x14_P2.54mm_Vertical, symbol Connector:Conn_01x14_Socket
- added J4: Conn_01x05_Socket, Connector_PinSocket_2.54mm:PinSocket_1x05_P2.54mm_Vertical, symbol Connector:Conn_01x05_Socket
- added VR16, VR17, VR18, VR19, VR20: T93YA104KT20, KiCad:T93YA5K10, symbol T93YA104KT20:T93YA104KT20
- C1, C2: footprint Connector_PinSocket_1.27mm:PinSocket_1x02_P1.27mm_Vertical -> Connector_PinSocket_2.54mm:PinSocket_1x02_P2.54mm_Vertical
- J23: footprint Connector_PinSocket_1.27mm:PinSocket_1x20_P1.27mm_Vertical -> Connector_PinSocket_2.54mm:PinSocket_1x20_P2.54mm_Vertical
Connections:
- net +5V: now also J2.1 (Pin_1), VR16.1 (A), VR16.2 (B), VR17.1 (A), VR17.2 (B), VR18.1 (A), VR18.2 (B), VR19.1 (A), VR19.2 (B), VR20.1 (A), VR20.2 (B)
- net A1: now also J3.4 (Pin_4)
- net A10: now also J4.5 (Pin_5)
- net A2: now also J3.5 (Pin_5)
- net A3: now also J3.6 (Pin_6)
- net A4: now also J3.7 (Pin_7)
- net A5: now also J3.8 (Pin_8)
- net A6: now also J4.1 (Pin_1)
- net A7: now also J4.2 (Pin_2)
- net A8: now also J4.3 (Pin_3)
- net A9: now also J4.4 (Pin_4)
- net GND: now also J2.4 (Pin_4); no longer U10.3 (NON-INV_INPUT), U6.3 (NON-INV_INPUT), U7.3 (NON-INV_INPUT), U8.3 (NON-INV_INPUT), U9.3 (NON-INV_INPUT)
- new net: U10.3 (NON-INV_INPUT), VR20.3 (C)
- new net: U9.3 (NON-INV_INPUT), VR19.3 (C)
- new net: U7.3 (NON-INV_INPUT), VR17.3 (C)
- new net: U8.3 (NON-INV_INPUT), VR18.3 (C)
- new net: U6.3 (NON-INV_INPUT), VR16.3 (C)
- no-connect marks 10 -> 31
Other:
- note added: "PCB P2I"
- moved on the sheet: J23
